File: seamal/seamal.sch (KiCad schematic (older format))
At the start: 17 parts, among them J1 Conn_01x02_Female, J2 Conn_01x03_Female, J3 Conn_01x02_Female, M1 Motor_DC, SW2 SW_DIP_x02, U1 STM32F303K8Tx, U2 BMX055, U3 DRV8830, U4 W25Q128JVS

Commit message: test1
Parts:
- added D?: LED, symbol Device:LED
Changed lines of the file:
@@
 $EndComp
 NoConn ~ 2250 2500
+$Comp
+L Device:LED D?
+U 1 1 6172A662
+P 7100 2650
+F 0 "D?" H 7093 2867 50  0000 C CNN
+F 1 "LED" H 7093 2776 50  0000 C CNN
+F 2 "" H 7100 2650 50  0001 C CNN
+F 3 "~" H 7100 2650 50  0001 C CNN
+	1    7100 2650
+	1    0    0    -1
+$EndComp
 $EndSCHEMATC
